File: schematics/output/sheets/SD1015_SD1525_sheet2.sch (EAGLE design)
At the start: 263 parts, among them U1A U1 section, pins 1/2/3 - DIFF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, U1B U1 section, pins 4/5/6/7/8, U2B U2 section - A.V. AMPLIFIER, U9B U9 section - ECC

Commit message: Fix transformer winding order, LOCKOUT's bottom pins, and label direction
Three defects reported off the Fusion render of sheet 8.

The transformer primary is drawn 3-2-1 down the coil, not 1-2-3 -- pin 3 is the
top terminal on the sheet. Listed the wrong way round, DRIVER pin 2 at the top
had to cross to T4 pin 3 at the bottom, and every driver-to-transformer lead
crossed its neighbours. That crossing was also what forced N_T3P3, N_T4P3 and
N_XFMR_CT to be declined for overlapping, which is why the centre-tap spine was
missing from the picture. With the order corrected all 15 transcribed nets draw
and nothing is declined.

LOCKOUT's two inhibit inputs come up from underneath on the drawing; they were
on the left because BLOCK had no bottom edge. BLOCK_SIDES gains "bottom" and
the symbol spreads those pins along the lower edge.

Net labels ran left to right from wherever they were anchored, so a label on a
stub pointing left read back over the part it belonged to -- which buried R95
and the transformer pins under their own net names. A label now reads away from
its pin.

Netlist untouched: 263 parts, 166 nets, 627 pin connections. Zero overlapping
wires on all nine sheets, 168 tests.

Co-Authored-By: Claude Opus 5 <noreply@anthropic.com>
Parts:
- T3: device sd1525:DS_XFMR_3 -> sd1525:DS_XFMR_4
Other:
- moved on the sheet: LOCKOUT
